Commit message: updated package m2wr with rviz launch and camera in there

File: m2wr/urdf/m2wr.urdf.xacro (robot description, xacro)
@@ -35,5 +35,6 @@
       <origin rpy="0 0 0" xyz="0 0 0"/>
       <geometry>
-        <box size="0.5 0.3 0.07"/>
+        <!--box size="0.5 0.3 0.07"/-->
+        <cylinder radius="0.05" length="0.1"/>
       </geometry>
       <material name="blue"/>
@@ -149,3 +150,63 @@
     </sensor>
   </gazebo>
+<gazebo reference="camera_link">
+<material>Gazebo/Green</material>
+<sensor type="camera" name="camera">
+<update_rate>30.0</update_rate>
+<visualize></visualize>
+<camera name="head">
+<horizontal_fov>1.3962634</horizontal_fov>
+<image>
+<width>800</width>
+<height>800</height>
+<format>R8G8B8</format>
+</image>
+<clip>
+<near>0.02</near>
+<far>300</far>
+</clip>
+</camera>
+<plugin name="camera_controller" filename="libgazebo_ros_camera.so">
+<alwaysOn>true</alwaysOn>
+<updateRate>0.0</updateRate>
+<cameraName>m2wr/camera</cameraName>
+<imageTopicName>image_raw</imageTopicName>
+<cameraInfoTopicName>camera_info</cameraInfoTopicName>
+<frameName>camera_link</frameName>
+<hackBaseline>0.07</hackBaseline>
+<distortionK1>0.0</distortionK1>
+<distortionK2>0.0</distortionK2>
+<distortionK3>0.0</distortionK3>
+<distortionT1>0.0</distortionT1>
+<distortionT2>0.0</distortionT2>
+</plugin>
+</sensor>
+</gazebo>
+<link name="camera_link">
+<collision>
+<origin xyz="0 0 0" rpy="0 0 0"/>
+<geometry>
+<box size="0.05 0.05 0.05"/>
+</geometry>
+</collision>
+<visual>
+<origin xyz="0 0 0" rpy="0 0 0"/>
+<geometry>
+<box size="0.05 0.05 0.05"/>
+</geometry>
+<material name="green"/>
+</visual>
+<inertial>
+<mass value="0.3" />
+<origin xyz="0 0 0" rpy="0 0 0"/>
+<box_inertia m="0.05" x="0.05" y="0.05" z="0.05" />
+<inertia ixx="1e-6" ixy="0" ixz="0" iyy="1e-6" iyz="0" izz="1e-6" />
+</inertial>
+</link>
+<joint name="camera_joint" type="fixed">
+<axis xyz="0 1 0" />
+<origin xyz=".25 0 0" rpy="0 0 0"/>
+<parent link="link_chassis"/>
+<child link="camera_link"/>
+</joint>
 </robot>
